File: hw/trunk/board_power.brd (EAGLE design)
At the start: 100 x 80 mm, 20 parts

Commit message: - Fixed missing wire VDD
git-svn-id: svn://192.168.1.40/net/garden@356 1a6b750e-079f-425f-90e7-3a118970be6b
Connections:
- removed net N$13: C2.+, C4.2, U$5.P$4
- net VCC: now also C2.+, C4.2, U$5.P$4
Routing:
- net VCC: track 90.2 -> 129.6 mm
- net N$13: track 13.1 -> 0.00 mm
Other:
- board size 100 x 80 mm -> 100 x 68.6 mm
Changed lines of the file:
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@@
 <grid distance="0.025" unitdist="inch" unit="inch" style="lines" multiple="1" display="no" altdistance="0.0125" altunitdist="inch" altunit="inch"/>
 <layers>
-<layer number="1" name="Top" color="4" fill="1" visible="no" active="yes"/>
-<layer number="16" name="Bottom" color="1" fill="1" visible="no" active="yes"/>
-<layer number="17" name="Pads" color="2" fill="1" visible="no" active="yes"/>
-<layer number="18" name="Vias" color="2" fill="1" visible="no" active="yes"/>
-<layer number="19" name="Unrouted" color="6" fill="1" visible="no" active="yes"/>
+<layer number="1" name="Top" color="4" fill="1" visible="yes" active="yes"/>
+<layer number="16" name="Bottom" color="1" fill="1" visible="yes" active="yes"/>
+<layer number="17" name="Pads" color="2" fill="1" visible="yes" active="yes"/>
+<layer number="18" name="Vias" color="2" fill="1" visible="yes" active="yes"/>
+<layer number="19" name="Unrouted" color="6" fill="1" visible="yes" active="yes"/>
 <layer number="20" name="Dimension" color="15" fill="1" visible="yes" active="yes"/>
 <layer number="21" name="tPlace" color="7" fill="1" visible="yes" active="yes"/>
-<layer number="22" name="bPlace" color="7" fill="1" visible="no" active="yes"/>
-<layer number="23" name="tOrigins" color="15" fill="1" visible="no" active="yes"/>
-<layer number="24" name="bOrigins" color="15" fill="1" visible="no" active="yes"/>
+<layer number="22" name="bPlace" color="7" fill="1" visible="yes" active="yes"/>
+<layer number="23" name="tOrigins" color="15" fill="1" visible="yes" active="yes"/>
+<layer number="24" name="bOrigins" color="15" fill="1" visible="yes" active="yes"/>
 <layer number="25" name="tNames" color="7" fill="1" visible="yes" active="yes"/>
-<layer number="26" name="bNames" color="7" fill="1" visible="no" active="yes"/>
-<layer number="27" name="tValues" color="7" fill="1" visible="no" active="yes"/>
-<layer number="28" name="bValues" color="7" fill="1" visible="no" active="yes"/>
-<layer number="29" name="tStop" color="7" fill="3" visible="no" active="yes"/>
-<layer number="30" name="bStop" color="7" fill="6" visible="no" active="yes"/>
-<layer number="31" name="tCream" color="7" fill="4" visible="no" active="yes"/>
-<layer number="32" name="bCream" color="7" fill="5" visible="no" active="yes"/>
-<layer number="33" name="tFinish" color="6" fill="3" visible="no" active="yes"/>
-<layer number="34" name="bFinish" color="6" fill="6" visible="no" active="yes"/>
-<layer number="35" name="tGlue" color="7" fill="4" visible="no" active="yes"/>
-<layer number="36" name="bGlue" color="7" fill="5" visible="no" active="yes"/>
-<layer number="37" name="tTest" color="7" fill="1" visible="no" active="yes"/>
-<layer number="38" name="bTest" color="7" fill="1" visible="no" active="yes"/>
-<layer number="39" name="tKeepout" color="4" fill="11" visible="no" active="yes"/>
-<layer number="40" name="bKeepout" color="1" fill="11" visible="no" active="yes"/>
-<layer number="41" name="tRestrict" color="4" fill="10" visible="no" active="yes"/>
-<layer number="42" name="bRestrict" color="1" fill="10" visible="no" active="yes"/>
-<layer number="43" name="vRestrict" color="2" fill="10" visible="no" active="yes"/>
-<layer number="44" name="Drills" color="7" fill="1" visible="no" active="yes"/>
-<layer number="45" name="Holes" color="7" fill="1" visible="no" active="yes"/>
-<layer number="46" name="Milling" color="3" fill="1" visible="no" active="yes"/>
-<layer number="47" name="Measures" color="7" fill="1" visible="no" active="yes"/>
-<layer number="48" name="Document" color="7" fill="1" visible="no" active="yes"/>
-<layer number="49" name="Reference" color="7" fill="1" visible="no" active="yes"/>
-<layer number="51" name="tDocu" color="7" fill="1" visible="no" active="yes"/>
-<layer number="52" name="bDocu" color="7" fill="1" visible="no" active="yes"/>
+<layer number="26" name="bNames" color="7" fill="1" visible="yes" active="yes"/>
+<layer number="27" name="tValues" color="7" fill="1" visible="yes" active="yes"/>
+<layer number="28" name="bValues" color="7" fill="1" visible="yes" active="yes"/>
+<layer number="29" name="tStop" color="7" fill="3" visible="yes" active="yes"/>
+<layer number="30" name="bStop" color="7" fill="6" visible="yes" active="yes"/>
+<layer number="31" name="tCream" color="7" fill="4" visible="yes" active="yes"/>
+<layer number="32" name="bCream" color="7" fill="5" visible="yes" active="yes"/>
+<layer number="33" name="tFinish" color="6" fill="3" visible="yes" active="yes"/>
+<layer number="34" name="bFinish" color="6" fill="6" visible="yes" active="yes"/>
+<layer number="35" name="tGlue" color="7" fill="4" visible="yes" active="yes"/>
+<layer number="36" name="bGlue" color="7" fill="5" visible="yes" active="yes"/>
+<layer number="37" name="tTest" color="7" fill="1" visible="yes" active="yes"/>
+<layer number="38" name="bTest" color="7" fill="1" visible="yes" active="yes"/>
+<layer number="39" name="tKeepout" color="4" fill="11" visible="yes" active="yes"/>
+<layer number="40" name="bKeepout" color="1" fill="11" visible="yes" active="yes"/>
+<layer number="41" name="tRestrict" color="4" fill="10" visible="yes" active="yes"/>
+<layer number="42" name="bRestrict" color="1" fill="10" visible="yes" active="yes"/>
+<layer number="43" name="vRestrict" color="2" fill="10" visible="yes" active="yes"/>
+<layer number="44" name="Drills" color="7" fill="1" visible="yes" active="yes"/>
+<layer number="45" name="Holes" color="7" fill="1" visible="yes" active="yes"/>
+<layer number="46" name="Milling" color="3" fill="1" visible="yes" active="yes"/>
+<layer number="47" name="Measures" color="7" fill="1" visible="yes" active="yes"/>
+<layer number="48" name="Document" color="7" fill="1" visible="yes" active="yes"/>
+<layer number="49" name="Reference" color="7" fill="1" visible="yes" active="yes"/>
+<layer number="51" name="tDocu" color="7" fill="1" visible="yes" active="yes"/>
+<layer number="52" name="bDocu" color="7" fill="1" visible="yes" active="yes"/>
 <layer number="90" name="Modules" color="5" fill="1" visible="no" active="no"/>
 <layer number="91" name="Nets" color="2" fill="1" visible="no" active="no"/>
@@
 <plain>
 <wire x1="0" y1="0" x2="100" y2="0" width="0" layer="20"/>
-<wire x1="100" y1="0" x2="100" y2="80" width="0" layer="20"/>
-<wire x1="100" y1="80" x2="0" y2="80" width="0" layer="20"/>
-<wire x1="0" y1="80" x2="0" y2="0" width="0" layer="20"/>
+<wire x1="100" y1="0" x2="100" y2="68.57" width="0" layer="20"/>
+<wire x1="100" y1="68.57" x2="0" y2="68.57" width="0" layer="20"/>
+<wire x1="0" y1="68.57" x2="0" y2="0" width="0" layer="20"/>
 <text x="18.415" y="57.785" size="1.778" layer="16" rot="MR0">LuxHardware
 NET-GARD
@@
 <via x="63.5" y="32.7025" extent="1-16" drill="1" diameter="0.8128" shape="octagon"/>
 <wire x1="63.5" y1="49.53" x2="63.5" y2="32.7025" width="0.6096" layer="1"/>
+<wire x1="63.5" y1="32.67" x2="61.31" y2="32.67" width="0.6096" layer="16"/>
+<wire x1="61.31" y1="32.67" x2="46.99" y2="46.99" width="0.6096" layer="16"/>
+<wire x1="46.99" y1="46.99" x2="43.18" y2="46.99" width="0.6096" layer="16"/>
+<contactref element="C2" pad="+"/>
+<contactref element="U$5" pad="P$4"/>
+<contactref element="C4" pad="2"/>
+<wire x1="44.8437" y1="44.8437" x2="44.8437" y2="39.3954" width="0.635" layer="16"/>
+<wire x1="43.18" y1="46.99" x2="44.8437" y2="44.8437" width="0.635" layer="16"/>
+<wire x1="44.8437" y1="39.3954" x2="44.45" y2="39.37" width="0.635" layer="16"/>
+<wire x1="43.18" y1="46.99" x2="40.64" y2="50.8" width="0.4064" layer="16"/>
 <wire x1="63.5" y1="49.53" x2="59.9313" y2="49.4538" width="0" layer="19" extent="16-16"/>
 <wire x1="63.5" y1="32.67" x2="63.5" y2="32.7025" width="0" layer="19" extent="16-16"/>
@@
 <wire x1="25.2284" y1="12.5284" x2="44.45" y2="31.75" width="0.6096" layer="16"/>
 </signal>
-<signal name="N$13">
-<contactref element="C2" pad="+"/>
-<contactref element="U$5" pad="P$4"/>
-<wire x1="44.8437" y1="44.8437" x2="44.8437" y2="39.3954" width="0.635" layer="16"/>
-<wire x1="43.18" y1="46.99" x2="44.8437" y2="44.8437" width="0.635" layer="16"/>
-<wire x1="44.8437" y1="39.3954" x2="44.45" y2="39.37" width="0.635" layer="16"/>
-<contactref element="C4" pad="2"/>
-<wire x1="43.18" y1="46.99" x2="40.64" y2="50.8" width="0.4064" layer="16"/>
-</signal>
 <signal name="N$15">
