File: hw/trunk/board_power.sch (EAGLE design)
At the start: 20 parts

Commit message: - Fixed missing wire VDD
git-svn-id: svn://192.168.1.40/net/garden@356 1a6b750e-079f-425f-90e7-3a118970be6b
Connections:
- removed net N$13: C2.+, C4.2, U$5.VOUT
- net VCC: now also C2.+, C4.2, U$5.VOUT
Changed lines of the file:
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@@
 <part name="H2" library="holes" deviceset="MOUNT-HOLE" device="3.6"/>
 <part name="H3" library="holes" deviceset="MOUNT-HOLE" device="3.6"/>
+<part name="P+3" library="supply1" deviceset="VCC" device=""/>
 </parts>
 <sheets>
@@
 <instance part="H2" gate="G$1" x="-40.64" y="127"/>
 <instance part="H3" gate="G$1" x="-27.94" y="127"/>
+<instance part="P+3" gate="VCC" x="-10.16" y="27.94"/>
 </instances>
 <busses>
@@
 <wire x1="15.24" y1="71.12" x2="15.24" y2="78.74" width="0.1524" layer="91"/>
 </segment>
+<segment>
+<pinref part="C2" gate="G$1" pin="+"/>
+<wire x1="-10.16" y1="17.78" x2="-10.16" y2="20.32" width="0.1524" layer="91"/>
+<pinref part="U$5" gate="G$1" pin="VOUT"/>
+<wire x1="-10.16" y1="20.32" x2="-12.7" y2="20.32" width="0.1524" layer="91"/>
+<wire x1="-5.08" y1="10.16" x2="-5.08" y2="20.32" width="0.1524" layer="91"/>
+<wire x1="-5.08" y1="20.32" x2="-10.16" y2="20.32" width="0.1524" layer="91"/>
+<junction x="-10.16" y="20.32"/>
+<pinref part="C4" gate="G$1" pin="2"/>
+<pinref part="P+3" gate="VCC" pin="VCC"/>
+<wire x1="-10.16" y1="20.32" x2="-10.16" y2="25.4" width="0.1524" layer="91"/>
+</segment>
 </net>
 <net name="N$1" class="0">
@@
 </segment>
 </net>
-<net name="N$13" class="0">
-<segment>
-<pinref part="C2" gate="G$1" pin="+"/>
-<wire x1="-10.16" y1="17.78" x2="-10.16" y2="20.32" width="0.1524" layer="91"/>
-<pinref part="U$5" gate="G$1" pin="VOUT"/>
-<wire x1="-10.16" y1="20.32" x2="-12.7" y2="20.32" width="0.1524" layer="91"/>
-<wire x1="-5.08" y1="10.16" x2="-5.08" y2="20.32" width="0.1524" layer="91"/>
-<wire x1="-5.08" y1="20.32" x2="-10.16" y2="20.32" width="0.1524" layer="91"/>
-<junction x="-10.16" y="20.32"/>
-<pinref part="C4" gate="G$1" pin="2"/>
-</segment>
-</net>
