File: trunk/mcu_board.brd (EAGLE design)
At the start: 132.1 x 55.5 mm, 41 parts, among them IC1 MCU-CARD-MIKROE, IC2 MAX485ST3485, IC3 78L05, J1 MAGJACK, J2 DATA-BUS, J3 POWER-IN, J4 POWER-BUS, Q1 BC546B, Q2 IRF9630

Commit message: ?
git-svn-id: svn://192.168.1.40/net/mcu@534 1a6b750e-079f-425f-90e7-3a118970be6b
Parts:
- added R10: 10k, custom:0207/10
Connections:
- net N$18 renamed 485_B
- net N$24 renamed 485_A
- net N$13: now also R10.2
- net VCC: now also R10.1
Changed lines of the file:
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@@
 <layer number="14" name="Route14" color="1" fill="6" visible="no" active="no"/>
 <layer number="15" name="Route15" color="4" fill="6" visible="no" active="no"/>
-<layer number="16" name="Bottom" color="1" fill="1" visible="no" active="yes"/>
-<layer number="17" name="Pads" color="2" fill="1" visible="no" active="yes"/>
-<layer number="18" name="Vias" color="2" fill="1" visible="no" active="yes"/>
-<layer number="19" name="Unrouted" color="6" fill="1" visible="no" active="yes"/>
+<layer number="16" name="Bottom" color="1" fill="1" visible="yes" active="yes"/>
+<layer number="17" name="Pads" color="2" fill="1" visible="yes" active="yes"/>
+<layer number="18" name="Vias" color="2" fill="1" visible="yes" active="yes"/>
+<layer number="19" name="Unrouted" color="6" fill="1" visible="yes" active="yes"/>
 <layer number="20" name="Dimension" color="15" fill="1" visible="yes" active="yes"/>
 <layer number="21" name="tPlace" color="7" fill="1" visible="yes" active="yes"/>
@@
 <attribute name="VALUE" x="86.0806" y="65.405" size="1.27" layer="27" ratio="10" rot="R180"/>
 </element>
+<element name="R10" library="custom" package="0207/10" value="10k" x="20.32" y="40.64"/>
 </elements>
 <signals>
@@
 <wire x1="45.72" y1="86.36" x2="52.07" y2="80.01" width="0.4064" layer="16"/>
 <wire x1="52.07" y1="80.01" x2="52.07" y2="77.47" width="0.4064" layer="16"/>
+<contactref element="R10" pad="1"/>
+<wire x1="15.24" y1="40.64" x2="40.29" y2="50.8" width="0" layer="19" extent="1-1"/>
 </signal>
 <signal name="GND">
@@
 <wire x1="48.9712" y1="72.1106" x2="48.9712" y2="76.9112" width="0.4064" layer="16"/>
 <wire x1="48.9712" y1="76.9112" x2="49.53" y2="77.47" width="0.4064" layer="16"/>
+<contactref element="R10" pad="2"/>
+<wire x1="25.4" y1="40.64" x2="48.9712" y2="72.1106" width="0" layer="19" extent="1-1"/>
 </signal>
 <signal name="N$14">
@@
 <wire x1="102.87" y1="67.31" x2="100.33" y2="69.85" width="0.4064" layer="16"/>
 </signal>
-<signal name="N$18">
+<signal name="485_B">
 <contactref element="J2" pad="1"/>
 <contactref element="IC2" pad="7"/>
@@
 <wire x1="65.405" y1="57.15" x2="65.405" y2="49.53" width="0.4064" layer="16"/>
 </signal>
-<signal name="N$24">
+<signal name="485_A">
 <contactref element="IC2" pad="6"/>
 <contactref element="J2" pad="2"/>
