File: trunk/mcu_board.sch (EAGLE design)
At the start: 41 parts, among them IC1 MCU-CARD-MIKROE, IC2 MAX485ST3485, IC3 78L05, J1 MAGJACK, J2 DATA-BUS, J3 POWER-IN, J4 POWER-BUS, Q1 BC546B, Q2 IRF9630

Commit message: ?
git-svn-id: svn://192.168.1.40/net/mcu@534 1a6b750e-079f-425f-90e7-3a118970be6b
Parts:
- added R10: 10k, custom:R-EU_0207/10
Connections:
- net N$18 renamed 485_B
- net N$24 renamed 485_A
- net N$13: now also R10.2
- net VCC: now also R10.1
Changed lines of the file:
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@@
 <part name="GND18" library="custom" deviceset="GND" device=""/>
 <part name="R9" library="custom" deviceset="R-EU_" device="0207/10" value="4k7"/>
+<part name="R10" library="custom" deviceset="R-EU_" device="0207/10" value="10k"/>
+<part name="P+1" library="custom" deviceset="VCC" device=""/>
 </parts>
 <sheets>
@@
 <instance part="GND18" gate="1" x="-53.34" y="-7.62"/>
 <instance part="R9" gate="G$1" x="-53.34" y="12.7" rot="R90"/>
+<instance part="R10" gate="G$1" x="2.54" y="111.76" rot="R180"/>
+<instance part="P+1" gate="VCC" x="10.16" y="116.84"/>
 </instances>
 <busses>
@@
 <junction x="-20.32" y="71.12"/>
 </segment>
+<segment>
+<pinref part="R10" gate="G$1" pin="1"/>
+<pinref part="P+1" gate="VCC" pin="VCC"/>
+<wire x1="7.62" y1="111.76" x2="10.16" y2="111.76" width="0.1524" layer="91"/>
+<wire x1="10.16" y1="111.76" x2="10.16" y2="114.3" width="0.1524" layer="91"/>
+</segment>
 </net>
 <net name="N$1" class="0">
@@
 <pinref part="U$1" gate="G$1" pin="/MCLR"/>
 <wire x1="-2.54" y1="93.98" x2="-35.56" y2="93.98" width="0.1524" layer="91"/>
-<wire x1="-5.08" y1="111.76" x2="-2.54" y2="109.22" width="0.1524" layer="91"/>
-<wire x1="-2.54" y1="109.22" x2="-2.54" y2="93.98" width="0.1524" layer="91"/>
+<wire x1="-5.08" y1="111.76" x2="-2.54" y2="111.76" width="0.1524" layer="91"/>
+<wire x1="-2.54" y1="111.76" x2="-2.54" y2="93.98" width="0.1524" layer="91"/>
 <junction x="-2.54" y="93.98"/>
 <pinref part="BUT1" gate="G$1" pin="1@A"/>
+<pinref part="R10" gate="G$1" pin="2"/>
+<junction x="-2.54" y="111.76"/>
 </segment>
 </net>
@@
 </segment>
 </net>
-<net name="N$18" class="0">
+<net name="485_B" class="0">
 <segment>
 <pinref part="J2" gate="G$1" pin="1"/>
@@
 </segment>
 </net>
-<net name="N$24" class="0">
+<net name="485_A" class="0">
 <segment>
 <pinref part="IC2" gate="G$1" pin="A"/>
