File: trunk/microbean.sch (EAGLE design)
At the start: 17 parts, among them IC2 MAX485ST3485, IC3 PIC16F1827SO

Commit message: - WIP
git-svn-id: svn://192.168.1.40/net/microbean@535 1a6b750e-079f-425f-90e7-3a118970be6b
Connections:
- removed net N$4: C2.1, C4.+, IC1.OUT, IC3.VDD, U$1.+VCC
- new net N$23: IC2G$1.DE, IC2G$1.RE/, IC3.RA1
- net N$12: no longer IC2G$1.DE, IC2G$1.RE/, IC3.RA1
- net N$13: now also C2.1, C4.+, IC1.OUT, IC3.VDD, U$1.+VCC

Commit message: WIP
git-svn-id: svn://192.168.1.40/net/microbean@537 1a6b750e-079f-425f-90e7-3a118970be6b
Parts:
- C3, C4: device custom:CPOL-EUE2-4 -> custom:CPOL-EUSMD4X5.3
- J3: device custom:M04 -> custom:M05PTH
- U$3: value LEDPLCC2 -> LED1206; device custom:LEDPLCC2 -> custom:LED1206
Connections:
- new net N$4: IC3.RA7/OSC1, J3.2
- net N$18: now also J3.5; no longer J3.4
- net N$19: now also J3.4; no longer J3.3
- net N$20: now also J3.3; no longer J3.2
Other:
- moved on the sheet: C2, D3, J1
Changed lines of the file:
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@@
 <?xml version="1.0" encoding="utf-8"?>
 <!DOCTYPE eagle SYSTEM "eagle.dtd">
-<eagle version="7.5.0">
+<eagle version="7.7.0">
 <drawing>
 <settings>
@@
 <part name="C1" library="custom" deviceset="C-EU" device="C0805"/>
 <part name="C2" library="custom" deviceset="C-EU" device="C0805"/>
-<part name="C3" library="custom" deviceset="CPOL-EU" device="E2-4"/>
-<part name="C4" library="custom" deviceset="CPOL-EU" device="E2-4"/>
+<part name="C3" library="custom" deviceset="CPOL-EU" device="SMD4X5.3"/>
+<part name="C4" library="custom" deviceset="CPOL-EU" device="SMD4X5.3"/>
 <part name="J2" library="custom" deviceset="M02-SCREW-3.5MM" device="3.5MM"/>
 <part name="IC2" library="custom" deviceset="MAX485" device="ST3485"/>
@@
 <part name="U$2" library="custom" deviceset="PUSH-BUTTON" device=""/>
 <part name="GND4" library="custom" deviceset="GND" device=""/>
-<part name="U$3" library="custom" deviceset="LED" device="PLCC2"/>
+<part name="U$3" library="custom" deviceset="LED" device="1206" value="LED1206"/>
 <part name="GND5" library="custom" deviceset="GND" device=""/>
 <part name="R1" library="custom" deviceset="R-EU_" device="R0805"/>
@@
 <part name="GND7" library="custom" deviceset="GND" device=""/>
 <part name="C5" library="custom" deviceset="C-EU" device="C0805"/>
-<part name="J3" library="custom" deviceset="M04" device=""/>
+<part name="J3" library="custom" deviceset="M05" device="PTH"/>
 <part name="J4" library="custom" deviceset="M04" device=""/>
 </parts>
@@
 <instances>
 <instance part="IC1" gate="1" x="25.4" y="73.66"/>
-<instance part="J1" gate="G$1" x="-7.62" y="71.12"/>
-<instance part="GND1" gate="1" x="0" y="66.04"/>
+<instance part="J1" gate="G$1" x="-15.24" y="71.12"/>
+<instance part="GND1" gate="1" x="-7.62" y="66.04"/>
 <instance part="GND2" gate="1" x="25.4" y="60.96"/>
-<instance part="D3" gate="G$1" x="5.08" y="73.66"/>
+<instance part="D3" gate="G$1" x="0" y="73.66"/>
 <instance part="C1" gate="G$1" x="15.24" y="71.12"/>
-<instance part="C2" gate="G$1" x="66.04" y="71.12"/>
+<instance part="C2" gate="G$1" x="60.96" y="71.12"/>
 <instance part="C3" gate="G$1" x="10.16" y="71.12"/>
 <instance part="C4" gate="G$1" x="38.1" y="71.12"/>
@@
 <instance part="GND5" gate="1" x="101.6" y="17.78"/>
 <instance part="R1" gate="G$1" x="101.6" y="35.56" rot="R90"/>
-<instance part="GND6" gate="1" x="66.04" y="63.5"/>
+<instance part="GND6" gate="1" x="60.96" y="63.5"/>
 <instance part="IC2" gate="P" x="-17.78" y="43.18"/>
 <instance part="GND7" gate="1" x="-17.78" y="33.02"/>
 <instance part="C5" gate="G$1" x="-27.94" y="43.18"/>
-<instance part="J3" gate="G$1" x="129.54" y="66.04" rot="R180"/>
+<instance part="J3" gate="G$1" x="129.54" y="68.58" rot="R180"/>
 <instance part="J4" gate="G$1" x="129.54" y="50.8" rot="R180"/>
 </instances>
@@
 <pinref part="GND1" gate="1" pin="GND"/>
 <pinref part="J1" gate="G$1" pin="1"/>
-<wire x1="0" y1="68.58" x2="0" y2="71.12" width="0.1524" layer="91"/>
+<wire x1="-7.62" y1="68.58" x2="-7.62" y2="71.12" width="0.1524" layer="91"/>
 </segment>
 <segment>
@@
 <pinref part="J1" gate="G$1" pin="2"/>
 <pinref part="D3" gate="G$1" pin="A"/>
-<wire x1="2.54" y1="73.66" x2="0" y2="73.66" width="0.1524" layer="91"/>
+<wire x1="-2.54" y1="73.66" x2="-7.62" y2="73.66" width="0.1524" layer="91"/>
 </segment>
 </net>
@@
 <pinref part="IC1" gate="1" pin="IN"/>
 <pinref part="D3" gate="G$1" pin="C"/>
-<wire x1="7.62" y1="73.66" x2="10.16" y2="73.66" width="0.1524" layer="91"/>
+<wire x1="2.54" y1="73.66" x2="10.16" y2="73.66" width="0.1524" layer="91"/>
 <pinref part="C1" gate="G$1" pin="1"/>
 <wire x1="10.16" y1="73.66" x2="15.24" y2="73.66" width="0.1524" layer="91"/>
@@
 <wire x1="33.02" y1="73.66" x2="38.1" y2="73.66" width="0.1524" layer="91"/>
 <pinref part="C4" gate="G$1" pin="+"/>
-<wire x1="38.1" y1="73.66" x2="50.8" y2="73.66" width="0.1524" layer="91"/>
+<wire x1="38.1" y1="73.66" x2="43.18" y2="73.66" width="0.1524" layer="91"/>
 <junction x="38.1" y="73.66"/>
 <pinref part="IC3" gate="G$1" pin="VDD"/>
-<wire x1="50.8" y1="73.66" x2="66.04" y2="73.66" width="0.1524" layer="91"/>
-<wire x1="71.12" y1="73.66" x2="66.04" y2="73.66" width="0.1524" layer="91"/>
+<wire x1="43.18" y1="73.66" x2="60.96" y2="73.66" width="0.1524" layer="91"/>
+<wire x1="71.12" y1="73.66" x2="60.96" y2="73.66" width="0.1524" layer="91"/>
 <pinref part="U$1" gate="G$1" pin="+VCC"/>
-<wire x1="63.5" y1="73.66" x2="66.04" y2="73.66" width="0.1524" layer="91"/>
+<wire x1="63.5" y1="73.66" x2="60.96" y2="73.66" width="0.1524" layer="91"/>
 <wire x1="60.96" y1="22.86" x2="63.5" y2="22.86" width="0.1524" layer="91"/>
 <wire x1="63.5" y1="22.86" x2="63.5" y2="73.66" width="0.1524" layer="91"/>
 <junction x="63.5" y="73.66"/>
-<junction x="66.04" y="73.66"/>
-<wire x1="-17.78" y1="55.88" x2="50.8" y2="55.88" width="0.1524" layer="91"/>
-<wire x1="50.8" y1="55.88" x2="50.8" y2="73.66" width="0.1524" layer="91"/>
-<junction x="50.8" y="73.66"/>
+<junction x="60.96" y="73.66"/>
+<wire x1="-17.78" y1="55.88" x2="43.18" y2="55.88" width="0.1524" layer="91"/>
+<wire x1="43.18" y1="55.88" x2="43.18" y2="73.66" width="0.1524" layer="91"/>
+<junction x="43.18" y="73.66"/>
 <junction x="-17.78" y="50.8"/>
 </segment>
@@
 <pinref part="IC3" gate="G$1" pin="RA2"/>
 <pinref part="J4" gate="G$1" pin="4"/>
-<wire x1="101.6" y1="45.72" x2="121.92" y2="45.72" width="0.1524" layer="91"/>
-<wire x1="121.92" y1="45.72" x2="121.92" y2="48.26" width="0.1524" layer="91"/>
+<wire x1="101.6" y1="45.72" x2="119.38" y2="45.72" width="0.1524" layer="91"/>
+<wire x1="121.92" y1="48.26" x2="119.38" y2="48.26" width="0.1524" layer="91"/>
+<wire x1="119.38" y1="48.26" x2="119.38" y2="45.72" width="0.1524" layer="91"/>
 </segment>
 </net>
@@
 <pinref part="IC3" gate="G$1" pin="RB1/RX"/>
 <wire x1="101.6" y1="58.42" x2="121.92" y2="58.42" width="0.1524" layer="91"/>
-<pinref part="J3" gate="G$1" pin="4"/>
 <wire x1="121.92" y1="58.42" x2="121.92" y2="63.5" width="0.1524" layer="91"/>
+<pinref part="J3" gate="G$1" pin="5"/>
 </segment>
 </net>
@@
 <wire x1="101.6" y1="63.5" x2="119.38" y2="63.5" width="0.1524" layer="91"/>
 <wire x1="119.38" y1="63.5" x2="119.38" y2="66.04" width="0.1524" layer="91"/>
-<pinref part="J3" gate="G$1" pin="3"/>
+<pinref part="J3" gate="G$1" pin="4"/>
 <wire x1="119.38" y1="66.04" x2="121.92" y2="66.04" width="0.1524" layer="91"/>
 </segment>
@@
 <wire x1="101.6" y1="66.04" x2="116.84" y2="66.04" width="0.1524" layer="91"/>
 <wire x1="116.84" y1="66.04" x2="116.84" y2="68.58" width="0.1524" layer="91"/>
-<pinref part="J3" gate="G$1" pin="2"/>
+<pinref part="J3" gate="G$1" pin="3"/>
 <wire x1="116.84" y1="68.58" x2="121.92" y2="68.58" width="0.1524" layer="91"/>
 </segment>
@@
 <segment>
 <pinref part="IC3" gate="G$1" pin="RA6/OSC2"/>
-<wire x1="71.12" y1="55.88" x2="68.58" y2="55.88" width="0.1524" layer="91"/>
-<wire x1="68.58" y1="55.88" x2="68.58" y2="78.74" width="0.1524" layer="91"/>
-<wire x1="68.58" y1="78.74" x2="119.38" y2="78.74" width="0.1524" layer="91"/>
-<wire x1="119.38" y1="78.74" x2="119.38" y2="71.12" width="0.1524" layer="91"/>
+<wire x1="71.12" y1="55.88" x2="66.04" y2="55.88" width="0.1524" layer="91"/>
+<wire x1="66.04" y1="55.88" x2="66.04" y2="81.28" width="0.1524" layer="91"/>
+<wire x1="66.04" y1="81.28" x2="119.38" y2="81.28" width="0.1524" layer="91"/>
+<wire x1="119.38" y1="81.28" x2="119.38" y2="73.66" width="0.1524" layer="91"/>
 <pinref part="J3" gate="G$1" pin="1"/>
-<wire x1="119.38" y1="71.12" x2="121.92" y2="71.12" width="0.1524" layer="91"/>
+<wire x1="121.92" y1="73.66" x2="119.38" y2="73.66" width="0.1524" layer="91"/>
 </segment>
 </net>
@@
 <pinref part="IC3" gate="G$1" pin="RA1"/>
 <wire x1="101.6" y1="43.18" x2="119.38" y2="43.18" width="0.1524" layer="91"/>
-<wire x1="119.38" y1="43.18" x2="119.38" y2="-7.62" width="0.1524" layer="91"/>
-<wire x1="119.38" y1="-7.62" x2="40.64" y2="-7.62" width="0.1524" layer="91"/>
+<wire x1="119.38" y1="43.18" x2="119.38" y2="-5.08" width="0.1524" layer="91"/>
+<wire x1="119.38" y1="-5.08" x2="40.64" y2="-5.08" width="0.1524" layer="91"/>
 <pinref part="IC2" gate="G$1" pin="DE"/>
 <wire x1="40.64" y1="40.64" x2="33.02" y2="40.64" width="0.1524" layer="91"/>
@@
 <pinref part="IC2" gate="G$1" pin="RE/"/>
 <wire x1="33.02" y1="35.56" x2="33.02" y2="40.64" width="0.1524" layer="91"/>
-<wire x1="40.64" y1="-7.62" x2="40.64" y2="40.64" width="0.1524" layer="91"/>
-</segment>
-</net>
+<wire x1="40.64" y1="-5.08" x2="40.64" y2="40.64" width="0.1524" layer="91"/>
+</segment>
+</net>
+<net name="N$4" class="0">
+<segment>
+<pinref part="IC3" gate="G$1" pin="RA7/OSC1"/>
+<wire x1="71.12" y1="58.42" x2="68.58" y2="58.42" width="0.1524" layer="91"/>
+<wire x1="68.58" y1="58.42" x2="68.58" y2="78.74" width="0.1524" layer="91"/>
+<wire x1="68.58" y1="78.74" x2="116.84" y2="78.74" width="0.1524" layer="91"/>
+<wire x1="116.84" y1="78.74" x2="116.84" y2="71.12" width="0.1524" layer="91"/>
+<pinref part="J3" gate="G$1" pin="2"/>
+<wire x1="116.84" y1="71.12" x2="121.92" y2="71.12" width="0.1524" layer="91"/>
+</segment>
+</net>
