File: microbean/microbean.sch (EAGLE design)
At the start: 17 parts, among them IC2 MAX485ST3485, IC3 PIC16F1827SO

Commit message: - WIP microbean for professional printing
git-svn-id: svn://mule/net/hardware/trunk@556 1a6b750e-079f-425f-90e7-3a118970be6b
Parts:
- added J5: (no value), custom:M02
Connections:
- net GND: now also J5.2
- net N$10: now also R1.2; no longer R1.1
- net N$13: now also J5.1
- net N$14: now also IC3.RB1/RX; no longer IC3.RA2
- net N$15: now also IC3.RB0; no longer IC3.RA3
- net N$17: now also IC3.RA3; no longer IC3.RB0
- net N$18: now also IC3.RA2; no longer IC3.RB1/RX
- net N$19: now also IC3.RA0; no longer IC3.RB3
- net N$20: now also IC3.RA7/OSC1; no longer IC3.RB4
- net N$21: now also IC3.RB4; no longer IC3.RA6/OSC2
- net N$4: now also IC3.RA6/OSC2; no longer IC3.RA7/OSC1
- net N$9: now also IC3.RB3, R1.1; no longer IC3.RA0, R1.2
Other:
- moved on the sheet: J3, J4
Changed lines of the file:
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@@
 <?xml version="1.0" encoding="utf-8"?>
 <!DOCTYPE eagle SYSTEM "eagle.dtd">
-<eagle version="7.7.0">
+<eagle version="7.5.0">
 <drawing>
 <settings>
@@
 <part name="J3" library="custom" deviceset="M05" device="PTH"/>
 <part name="J4" library="custom" deviceset="M04" device=""/>
+<part name="J5" library="custom" deviceset="M02" device=""/>
+<part name="GND8" library="custom" deviceset="GND" device=""/>
 </parts>
 <sheets>
@@
 <instance part="GND7" gate="1" x="-17.78" y="33.02"/>
 <instance part="C5" gate="G$1" x="-27.94" y="43.18"/>
-<instance part="J3" gate="G$1" x="129.54" y="68.58" rot="R180"/>
-<instance part="J4" gate="G$1" x="129.54" y="50.8" rot="R180"/>
+<instance part="J3" gate="G$1" x="137.16" y="68.58" rot="R180"/>
+<instance part="J4" gate="G$1" x="137.16" y="53.34" rot="MR0"/>
+<instance part="J5" gate="G$1" x="55.88" y="83.82" rot="R180"/>
+<instance part="GND8" gate="1" x="48.26" y="78.74"/>
 </instances>
 <busses>
@@
 <junction x="-17.78" y="35.56"/>
 </segment>
+<segment>
+<pinref part="J5" gate="G$1" pin="2"/>
+<pinref part="GND8" gate="1" pin="GND"/>
+</segment>
 </net>
 <net name="N$1" class="0">
@@
 <net name="N$9" class="0">
 <segment>
-<pinref part="IC3" gate="G$1" pin="RA0"/>
+<pinref part="IC3" gate="G$1" pin="RB3"/>
+<pinref part="R1" gate="G$1" pin="1"/>
+<wire x1="101.6" y1="30.48" x2="101.6" y2="63.5" width="0.1524" layer="91"/>
+</segment>
+</net>
+<net name="N$10" class="0">
+<segment>
 <pinref part="R1" gate="G$1" pin="2"/>
-</segment>
-</net>
-<net name="N$10" class="0">
-<segment>
-<pinref part="R1" gate="G$1" pin="1"/>
 <pinref part="U$3" gate="G$1" pin="A"/>
+<wire x1="101.6" y1="30.48" x2="101.6" y2="40.64" width="0.1524" layer="91"/>
 </segment>
 </net>
@@
 <junction x="43.18" y="73.66"/>
 <junction x="-17.78" y="50.8"/>
+<pinref part="J5" gate="G$1" pin="1"/>
+<wire x1="48.26" y1="83.82" x2="43.18" y2="83.82" width="0.1524" layer="91"/>
+<wire x1="43.18" y1="83.82" x2="43.18" y2="73.66" width="0.1524" layer="91"/>
 </segment>
 </net>
 <net name="N$14" class="0">
 <segment>
+<pinref part="IC3" gate="G$1" pin="RB1/RX"/>
+<pinref part="J4" gate="G$1" pin="4"/>
+<wire x1="101.6" y1="58.42" x2="104.14" y2="58.42" width="0.1524" layer="91"/>
+<wire x1="129.54" y1="55.88" x2="106.68" y2="55.88" width="0.1524" layer="91"/>
+<wire x1="106.68" y1="55.88" x2="106.68" y2="58.42" width="0.1524" layer="91"/>
+<wire x1="106.68" y1="58.42" x2="104.14" y2="58.42" width="0.1524" layer="91"/>
+</segment>
+</net>
+<net name="N$15" class="0">
+<segment>
+<pinref part="IC3" gate="G$1" pin="RB0"/>
+<wire x1="101.6" y1="55.88" x2="104.14" y2="55.88" width="0.1524" layer="91"/>
+<wire x1="104.14" y1="55.88" x2="104.14" y2="53.34" width="0.1524" layer="91"/>
+<wire x1="104.14" y1="53.34" x2="124.46" y2="53.34" width="0.1524" layer="91"/>
+<pinref part="J4" gate="G$1" pin="3"/>
+<wire x1="124.46" y1="53.34" x2="129.54" y2="53.34" width="0.1524" layer="91"/>
+</segment>
+</net>
+<net name="N$16" class="0">
+<segment>
+<pinref part="IC3" gate="G$1" pin="T0CKI/RA4"/>
+<pinref part="J4" gate="G$1" pin="2"/>
+<wire x1="101.6" y1="50.8" x2="129.54" y2="50.8" width="0.1524" layer="91"/>
+</segment>
+</net>
+<net name="N$17" class="0">
+<segment>
+<pinref part="IC3" gate="G$1" pin="RA3"/>
+<pinref part="J4" gate="G$1" pin="1"/>
+<wire x1="101.6" y1="48.26" x2="129.54" y2="48.26" width="0.1524" layer="91"/>
+</segment>
+</net>
+<net name="N$18" class="0">
+<segment>
 <pinref part="IC3" gate="G$1" pin="RA2"/>
-<pinref part="J4" gate="G$1" pin="4"/>
-<wire x1="101.6" y1="45.72" x2="119.38" y2="45.72" width="0.1524" layer="91"/>
-<wire x1="121.92" y1="48.26" x2="119.38" y2="48.26" width="0.1524" layer="91"/>
-<wire x1="119.38" y1="48.26" x2="119.38" y2="45.72" width="0.1524" layer="91"/>
-</segment>
-</net>
-<net name="N$15" class="0">
-<segment>
-<pinref part="IC3" gate="G$1" pin="RA3"/>
-<wire x1="101.6" y1="48.26" x2="106.68" y2="48.26" width="0.1524" layer="91"/>
-<wire x1="106.68" y1="48.26" x2="106.68" y2="50.8" width="0.1524" layer="91"/>
-<pinref part="J4" gate="G$1" pin="3"/>
-<wire x1="106.68" y1="50.8" x2="121.92" y2="50.8" width="0.1524" layer="91"/>
-</segment>
-</net>
-<net name="N$16" class="0">
-<segment>
-<pinref part="IC3" gate="G$1" pin="T0CKI/RA4"/>
-<wire x1="101.6" y1="50.8" x2="104.14" y2="50.8" width="0.1524" layer="91"/>
-<wire x1="104.14" y1="50.8" x2="104.14" y2="53.34" width="0.1524" layer="91"/>
-<pinref part="J4" gate="G$1" pin="2"/>
-<wire x1="104.14" y1="53.34" x2="121.92" y2="53.34" width="0.1524" layer="91"/>
-</segment>
-</net>
-<net name="N$17" class="0">
-<segment>
-<pinref part="IC3" gate="G$1" pin="RB0"/>
-<pinref part="J4" gate="G$1" pin="1"/>
-<wire x1="101.6" y1="55.88" x2="121.92" y2="55.88" width="0.1524" layer="91"/>
-</segment>
-</net>
-<net name="N$18" class="0">
-<segment>
-<pinref part="IC3" gate="G$1" pin="RB1/RX"/>
-<wire x1="101.6" y1="58.42" x2="121.92" y2="58.42" width="0.1524" layer="91"/>
-<wire x1="121.92" y1="58.42" x2="121.92" y2="63.5" width="0.1524" layer="91"/>
+<wire x1="101.6" y1="45.72" x2="121.92" y2="45.72" width="0.1524" layer="91"/>
+<wire x1="121.92" y1="45.72" x2="121.92" y2="63.5" width="0.1524" layer="91"/>
+<wire x1="121.92" y1="63.5" x2="129.54" y2="63.5" width="0.1524" layer="91"/>
 <pinref part="J3" gate="G$1" pin="5"/>
 </segment>
@@
 <net name="N$19" class="0">
 <segment>
-<pinref part="IC3" gate="G$1" pin="RB3"/>
-<wire x1="101.6" y1="63.5" x2="119.38" y2="63.5" width="0.1524" layer="91"/>
-<wire x1="119.38" y1="63.5" x2="119.38" y2="66.04" width="0.1524" layer="91"/>
+<pinref part="IC3" gate="G$1" pin="RA0"/>
+<wire x1="101.6" y1="40.64" x2="124.46" y2="40.64" width="0.1524" layer="91"/>
+<wire x1="124.46" y1="40.64" x2="124.46" y2="66.04" width="0.1524" layer="91"/>
 <pinref part="J3" gate="G$1" pin="4"/>
-<wire x1="119.38" y1="66.04" x2="121.92" y2="66.04" width="0.1524" layer="91"/>
+<wire x1="124.46" y1="66.04" x2="129.54" y2="66.04" width="0.1524" layer="91"/>
 </segment>
 </net>
 <net name="N$20" class="0">
 <segment>
+<pinref part="IC3" gate="G$1" pin="RA7/OSC1"/>
+<wire x1="71.12" y1="58.42" x2="71.12" y2="78.74" width="0.1524" layer="91"/>
+<wire x1="71.12" y1="78.74" x2="119.38" y2="78.74" width="0.1524" layer="91"/>
+<wire x1="119.38" y1="78.74" x2="119.38" y2="68.58" width="0.1524" layer="91"/>
+<pinref part="J3" gate="G$1" pin="3"/>
+<wire x1="119.38" y1="68.58" x2="129.54" y2="68.58" width="0.1524" layer="91"/>
+</segment>
+</net>
+<net name="N$21" class="0">
+<segment>
 <pinref part="IC3" gate="G$1" pin="RB4"/>
-<wire x1="101.6" y1="66.04" x2="116.84" y2="66.04" width="0.1524" layer="91"/>
-<wire x1="116.84" y1="66.04" x2="116.84" y2="68.58" width="0.1524" layer="91"/>
-<pinref part="J3" gate="G$1" pin="3"/>
-<wire x1="116.84" y1="68.58" x2="121.92" y2="68.58" width="0.1524" layer="91"/>
-</segment>
-</net>
-<net name="N$21" class="0">
-<segment>
-<pinref part="IC3" gate="G$1" pin="RA6/OSC2"/>
-<wire x1="71.12" y1="55.88" x2="66.04" y2="55.88" width="0.1524" layer="91"/>
-<wire x1="66.04" y1="55.88" x2="66.04" y2="81.28" width="0.1524" layer="91"/>
-<wire x1="66.04" y1="81.28" x2="119.38" y2="81.28" width="0.1524" layer="91"/>
-<wire x1="119.38" y1="81.28" x2="119.38" y2="73.66" width="0.1524" layer="91"/>
+<wire x1="101.6" y1="66.04" x2="104.14" y2="66.04" width="0.1524" layer="91"/>
+<wire x1="104.14" y1="66.04" x2="104.14" y2="83.82" width="0.1524" layer="91"/>
+<wire x1="104.14" y1="83.82" x2="124.46" y2="83.82" width="0.1524" layer="91"/>
+<wire x1="124.46" y1="83.82" x2="124.46" y2="73.66" width="0.1524" layer="91"/>
 <pinref part="J3" gate="G$1" pin="1"/>
-<wire x1="121.92" y1="73.66" x2="119.38" y2="73.66" width="0.1524" layer="91"/>
+<wire x1="129.54" y1="73.66" x2="124.46" y2="73.66" width="0.1524" layer="91"/>
 </segment>
 </net>
@@
 <net name="N$4" class="0">
 <segment>
-<pinref part="IC3" gate="G$1" pin="RA7/OSC1"/>
-<wire x1="71.12" y1="58.42" x2="68.58" y2="58.42" width="0.1524" layer="91"/>
-<wire x1="68.58" y1="58.42" x2="68.58" y2="78.74" width="0.1524" layer="91"/>
-<wire x1="68.58" y1="78.74" x2="116.84" y2="78.74" width="0.1524" layer="91"/>
-<wire x1="116.84" y1="78.74" x2="116.84" y2="71.12" width="0.1524" layer="91"/>
+<pinref part="IC3" gate="G$1" pin="RA6/OSC2"/>
+<wire x1="71.12" y1="55.88" x2="68.58" y2="55.88" width="0.1524" layer="91"/>
+<wire x1="68.58" y1="55.88" x2="68.58" y2="81.28" width="0.1524" layer="91"/>
+<wire x1="68.58" y1="81.28" x2="121.92" y2="81.28" width="0.1524" layer="91"/>
+<wire x1="121.92" y1="81.28" x2="121.92" y2="71.12" width="0.1524" layer="91"/>
 <pinref part="J3" gate="G$1" pin="2"/>
-<wire x1="116.84" y1="71.12" x2="121.92" y2="71.12" width="0.1524" layer="91"/>
-</segment>
-</net>
+<wire x1="121.92" y1="71.12" x2="129.54" y2="71.12" width="0.1524" layer="91"/>
+</segment>
+</net>

Commit message: - WIP, DRU finished
git-svn-id: svn://mule/net/hardware/trunk@557 1a6b750e-079f-425f-90e7-3a118970be6b
Parts:
- renumbered U$1 to ICSP, U$3 to D2
Connections:
- net N$13 renamed VCC
- net N$14 renamed RB1
- net N$15 renamed RB0
- net N$16 renamed RA4
- net N$17 renamed RA3
- net N$18 renamed RA2
- net N$19 renamed RA0
- net N$20 renamed RA7
- net N$21 renamed RB4
- net N$3 renamed B
- net N$4 renamed RA6
- net N$5 renamed A
- net N$6 renamed MCLR
- net N$7 renamed DAT
- net N$8 renamed CLK
Changed lines of the file:
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@@
 <part name="IC3" library="custom" deviceset="PIC16F1827" device="SO"/>
 <part name="GND3" library="custom" deviceset="GND" device=""/>
-<part name="U$1" library="custom" deviceset="ICSP-HEADER-5" device=""/>
+<part name="ICSP" library="custom" deviceset="ICSP-HEADER-5" device=""/>
 <part name="U$2" library="custom" deviceset="PUSH-BUTTON" device=""/>
 <part name="GND4" library="custom" deviceset="GND" device=""/>
-<part name="U$3" library="custom" deviceset="LED" device="1206" value="LED1206"/>
+<part name="D2" library="custom" deviceset="LED" device="1206" value="LED1206"/>
 <part name="GND5" library="custom" deviceset="GND" device=""/>
 <part name="R1" library="custom" deviceset="R-EU_" device="R0805"/>
@@
 <instance part="IC3" gate="G$1" x="88.9" y="58.42"/>
 <instance part="GND3" gate="1" x="68.58" y="17.78"/>
-<instance part="U$1" gate="G$1" x="53.34" y="20.32"/>
+<instance part="ICSP" gate="G$1" x="53.34" y="20.32"/>
 <instance part="U$2" gate="G$1" x="50.8" y="45.72" rot="R90"/>
 <instance part="GND4" gate="1" x="50.8" y="38.1"/>
-<instance part="U$3" gate="G$1" x="101.6" y="25.4"/>
+<instance part="D2" gate="G$1" x="101.6" y="25.4"/>
 <instance part="GND5" gate="1" x="101.6" y="17.78"/>
 <instance part="R1" gate="G$1" x="101.6" y="35.56" rot="R90"/>
@@
 <wire x1="71.12" y1="40.64" x2="68.58" y2="40.64" width="0.1524" layer="91"/>
 <wire x1="68.58" y1="40.64" x2="68.58" y2="20.32" width="0.1524" layer="91"/>
-<pinref part="U$1" gate="G$1" pin="GND"/>
+<pinref part="ICSP" gate="G$1" pin="GND"/>
 <wire x1="60.96" y1="20.32" x2="68.58" y2="20.32" width="0.1524" layer="91"/>
 <junction x="68.58" y="20.32"/>
@@
 </segment>
 <segment>
-<pinref part="U$3" gate="G$1" pin="K"/>
+<pinref part="D2" gate="G$1" pin="K"/>
 <pinref part="GND5" gate="1" pin="GND"/>
 </segment>
@@
 </segment>
 </net>
-<net name="N$3" class="0">
+<net name="B" class="0">
 <segment>
 <pinref part="J2" gate="G$1" pin="1"/>
@@
 </segment>
 </net>
-<net name="N$5" class="0">
+<net name="A" class="0">
 <segment>
 <pinref part="J2" gate="G$1" pin="2"/>
@@
 </segment>
 </net>
-<net name="N$6" class="0">
-<segment>
-<pinref part="U$1" gate="G$1" pin="/MCLR"/>
+<net name="MCLR" class="0">
+<segment>
+<pinref part="ICSP" gate="G$1" pin="/MCLR"/>
 <wire x1="60.96" y1="25.4" x2="60.96" y2="53.34" width="0.1524" layer="91"/>
 <pinref part="IC3" gate="G$1" pin="RA5/!MCLR"/>
@@
 </segment>
 </net>
-<net name="N$7" class="0">
+<net name="DAT" class="0">
 <segment>
 <pinref part="IC3" gate="G$1" pin="RB7/ICSPDAT"/>
@@
 <wire x1="109.22" y1="10.16" x2="63.5" y2="10.16" width="0.1524" layer="91"/>
 <wire x1="63.5" y1="10.16" x2="63.5" y2="17.78" width="0.1524" layer="91"/>
-<pinref part="U$1" gate="G$1" pin="DAT"/>
+<pinref part="ICSP" gate="G$1" pin="DAT"/>
 <wire x1="63.5" y1="17.78" x2="60.96" y2="17.78" width="0.1524" layer="91"/>
 </segment>
 </net>
-<net name="N$8" class="0">
-<segment>
-<pinref part="U$1" gate="G$1" pin="CLK"/>
+<net name="CLK" class="0">
+<segment>
+<pinref part="ICSP" gate="G$1" pin="CLK"/>
 <wire x1="60.96" y1="15.24" x2="60.96" y2="7.62" width="0.1524" layer="91"/>
 <wire x1="60.96" y1="7.62" x2="111.76" y2="7.62" width="0.1524" layer="91"/>
@@
 <segment>
 <pinref part="R1" gate="G$1" pin="2"/>
-<pinref part="U$3" gate="G$1" pin="A"/>
+<pinref part="D2" gate="G$1" pin="A"/>
 <wire x1="101.6" y1="30.48" x2="101.6" y2="40.64" width="0.1524" layer="91"/>
 </segment>
@@
 </segment>
 </net>
-<net name="N$13" class="0">
+<net name="VCC" class="0">
 <segment>
 <pinref part="C5" gate="G$1" pin="1"/>
@@
 <wire x1="43.18" y1="73.66" x2="60.96" y2="73.66" width="0.1524" layer="91"/>
 <wire x1="71.12" y1="73.66" x2="60.96" y2="73.66" width="0.1524" layer="91"/>
-<pinref part="U$1" gate="G$1" pin="+VCC"/>
+<pinref part="ICSP" gate="G$1" pin="+VCC"/>
 <wire x1="63.5" y1="73.66" x2="60.96" y2="73.66" width="0.1524" layer="91"/>
 <wire x1="60.96" y1="22.86" x2="63.5" y2="22.86" width="0.1524" layer="91"/>
@@
 </segment>
 </net>
-<net name="N$14" class="0">
+<net name="RB1" class="0">
 <segment>
 <pinref part="IC3" gate="G$1" pin="RB1/RX"/>
@@
 </segment>
 </net>
-<net name="N$15" class="0">
+<net name="RB0" class="0">
 <segment>
 <pinref part="IC3" gate="G$1" pin="RB0"/>
@@
 </segment>
 </net>
-<net name="N$16" class="0">
+<net name="RA4" class="0">
 <segment>
 <pinref part="IC3" gate="G$1" pin="T0CKI/RA4"/>
@@
 </segment>
 </net>
-<net name="N$17" class="0">
+<net name="RA3" class="0">
 <segment>
 <pinref part="IC3" gate="G$1" pin="RA3"/>
@@
 </segment>
 </net>
-<net name="N$18" class="0">
+<net name="RA2" class="0">
 <segment>
 <pinref part="IC3" gate="G$1" pin="RA2"/>
@@
 </segment>
 </net>
-<net name="N$19" class="0">
+<net name="RA0" class="0">
 <segment>
 <pinref part="IC3" gate="G$1" pin="RA0"/>
@@
 </segment>
 </net>
-<net name="N$20" class="0">
+<net name="RA7" class="0">
 <segment>
 <pinref part="IC3" gate="G$1" pin="RA7/OSC1"/>
@@
 </segment>
 </net>
-<net name="N$21" class="0">
+<net name="RB4" class="0">
 <segment>
 <pinref part="IC3" gate="G$1" pin="RB4"/>
@@
 </segment>
 </net>
-<net name="N$4" class="0">
+<net name="RA6" class="0">
 <segment>
 <pinref part="IC3" gate="G$1" pin="RA6/OSC2"/>

Commit message: - Refinements
git-svn-id: svn://mule/net/hardware/trunk@560 1a6b750e-079f-425f-90e7-3a118970be6b
Parts:
- C1, C2, C5: value (none) -> 100n
- C3, C4: value (none) -> 10u
- D3: value S1M -> S1A
- IC1: value (none) -> L78L33/L78L05
- IC2: value MAX485ST3485 -> ST485/ST3485
- R1: value (none) -> 560
Other:
- moved on the sheet: R1
Changed lines of the file:
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@@
 </classes>
 <parts>
-<part name="IC1" library="custom" deviceset="78LXX" device="SOT89"/>
+<part name="IC1" library="custom" deviceset="78LXX" device="SOT89" value="L78L33/L78L05"/>
 <part name="J1" library="custom" deviceset="M02-SCREW-3.5MM" device="3.5MM"/>
 <part name="GND1" library="custom" deviceset="GND" device=""/>
 <part name="GND2" library="custom" deviceset="GND" device=""/>
-<part name="D3" library="diode" deviceset="S1M" device=""/>
-<part name="C1" library="custom" deviceset="C-EU" device="C0805"/>
-<part name="C2" library="custom" deviceset="C-EU" device="C0805"/>
-<part name="C3" library="custom" deviceset="CPOL-EU" device="SMD4X5.3"/>
-<part name="C4" library="custom" deviceset="CPOL-EU" device="SMD4X5.3"/>
+<part name="D3" library="diode" deviceset="S1M" device="" value="S1A"/>
+<part name="C1" library="custom" deviceset="C-EU" device="C0805" value="100n"/>
+<part name="C2" library="custom" deviceset="C-EU" device="C0805" value="100n"/>
+<part name="C3" library="custom" deviceset="CPOL-EU" device="SMD4X5.3" value="10u"/>
+<part name="C4" library="custom" deviceset="CPOL-EU" device="SMD4X5.3" value="10u"/>
 <part name="J2" library="custom" deviceset="M02-SCREW-3.5MM" device="3.5MM"/>
-<part name="IC2" library="custom" deviceset="MAX485" device="ST3485"/>
+<part name="IC2" library="custom" deviceset="MAX485" device="ST3485" value="ST485/ST3485"/>
 <part name="IC3" library="custom" deviceset="PIC16F1827" device="SO"/>
 <part name="GND3" library="custom" deviceset="GND" device=""/>
@@
 <part name="D2" library="custom" deviceset="LED" device="1206" value="LED1206"/>
 <part name="GND5" library="custom" deviceset="GND" device=""/>
-<part name="R1" library="custom" deviceset="R-EU_" device="R0805"/>
+<part name="R1" library="custom" deviceset="R-EU_" device="R0805" value="560"/>
 <part name="GND6" library="custom" deviceset="GND" device=""/>
 <part name="GND7" library="custom" deviceset="GND" device=""/>
-<part name="C5" library="custom" deviceset="C-EU" device="C0805"/>
+<part name="C5" library="custom" deviceset="C-EU" device="C0805" value="100n"/>
 <part name="J3" library="custom" deviceset="M05" device="PTH"/>
 <part name="J4" library="custom" deviceset="M04" device=""/>
@@
 <instance part="D2" gate="G$1" x="101.6" y="25.4"/>
 <instance part="GND5" gate="1" x="101.6" y="17.78"/>
-<instance part="R1" gate="G$1" x="101.6" y="35.56" rot="R90"/>
+<instance part="R1" gate="G$1" x="101.6" y="33.02" rot="R270"/>
 <instance part="GND6" gate="1" x="60.96" y="63.5"/>
 <instance part="IC2" gate="P" x="-17.78" y="43.18"/>
@@
 <pinref part="IC3" gate="G$1" pin="RB3"/>
 <pinref part="R1" gate="G$1" pin="1"/>
-<wire x1="101.6" y1="30.48" x2="101.6" y2="63.5" width="0.1524" layer="91"/>
+<wire x1="101.6" y1="38.1" x2="101.6" y2="63.5" width="0.1524" layer="91"/>
 </segment>
 </net>
@@
 <pinref part="R1" gate="G$1" pin="2"/>
 <pinref part="D2" gate="G$1" pin="A"/>
-<wire x1="101.6" y1="30.48" x2="101.6" y2="40.64" width="0.1524" layer="91"/>
-</segment>
-</net>
+<wire x1="101.6" y1="27.94" x2="101.6" y2="30.48" width="0.1524" layer="91"/>
+</segment>
+</net>

Commit message: - Finishing up for quoting
git-svn-id: svn://mule/net/hardware/trunk@564 1a6b750e-079f-425f-90e7-3a118970be6b
Parts:
- added J6: (no value), custom:M02
- IC3: value PIC16F1827SO -> PIC16F1827SO18; device custom:PIC16F1827SO -> custom:PIC16F1827SO18
Connections:
- net N$11 renamed RB5
- net N$12 renamed RB2
- removed net CLK: IC3.RB6/ICSPCLK, ICSP.CLK
- removed net DAT: IC3.RB7/ICSPDAT, ICSP.DAT
- removed net RA6: IC3.RA6/OSC2, J3.2
- removed net RA7: IC3.RA7/OSC1, J3.3
- new net RA1: IC3.RA1, J3.2
- new net RB3: IC3.RB3, J3.4
- new net RB6: IC3.RB6/ICSPCLK, ICSP.CLK, J6.2
- new net RB7: IC3.RB7/ICSPDAT, ICSP.DAT, J6.1
- net N$23: now also IC3.RA6/OSC2; no longer IC3.RA1
- net N$9: now also IC3.RA7/OSC1; no longer IC3.RB3
- net RA0: now also J3.3; no longer J3.4
Other:
- moved on the sheet: C2, D2, R1
